File: Textier/pypad.kicad_pcb (KiCad board)
At the start: 2 copper layers, 100 x 100 mm, 76 parts, among them J1 Conn_01x05_Male, J2 Conn_01x03_Male, K1 SW_SPST, K10 SW_SPST, K11 SW_SPST, K12 SW_SPST, K13 SW_SPST, K14 SW_SPST, K15 SW_SPST, K16 SW_SPST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

Commit message: Feedback fixes
 - OSHW logo + github text
 - removed some leftover silkscreen
Parts:
- removed the REF** at (115.3, 35.4)
- added REF**: OSHW-Symbol_8.9x8mm_SilkScreen, Symbol:OSHW-Symbol_8.9x8mm_SilkScreen, B.Cu at (114.9, 35.6)
